File: SeeMMC.kicad_pcb (KiCad board)
At the start: 2 copper layers, 24 x 32 mm, 17 parts, among them J1 SD_Card, U1 TXS02612RTWR, U2 TPS7A1118PDRV

Commit message: Production ready
Other:
- board text added: "JLCJLCJLCJLC"
Changed lines of the file:
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@@
   (gr_arc (start 148.6 95.3) (mid 148.246447 95.153553) (end 148.1 94.8)
     (stroke (width 0.15) (type default)) (layer "Margin"))
+  (gr_text "JLCJLCJLCJLC" (at 149.75 79.6 90) (layer "B.SilkS")
+    (effects (font (size 0.9 0.9) (thickness 0.15) bold) (justify left bottom mirror))
+  )
   (gr_text "SeeMMC" (at 155.560715 68.9) (layer "F.SilkS")
     (effects (font (size 1.5 1.5) (thickness 0.2)) (justify left bottom))
@@
   (via (at 160.1 75.35) (size 0.45) (drill 0.2) (layers "F.Cu" "B.Cu") (free) (net 2))
   (via (at 162.65 81.8) (size 0.45) (drill 0.2) (layers "F.Cu" "B.Cu") (free) (net 2))
-  (via (at 149.8 82.35) (size 0.45) (drill 0.2) (layers "F.Cu" "B.Cu") (free) (net 2))
+  (via (at 150.15 82.35) (size 0.45) (drill 0.2) (layers "F.Cu" "B.Cu") (free) (net 2))
   (via (at 149.5 72) (size 0.45) (drill 0.2) (layers "F.Cu" "B.Cu") (free) (net 2))
   (via (at 160.1 94.45) (size 0.45) (drill 0.2) (layers "F.Cu" "B.Cu") (free) (net 2))
